File: adapter/.history/adapter.kicad_sch (KiCad schematic)
At the start: 17 parts, among them J1 USB_C_Receptacle_PowerOnly_6P, J2 Conn_01x06_Socket, J3 Conn_01x05_Socket, Q1 BC817, Q2 BC817, U1 NCP1117-3.3_SOT223

Commit message: schematic apdated
Parts:
- added R10, R9: 5.1k, symbol Device:R
- R5, R6: value 510 -> 5.1k
Connections:
- net +3.3V: now also R10.1, R9.1
- net SCL: now also R10.2
- net SDA: now also R9.2
